File: hardware/LocalCam1.kicad_pcb (KiCad board)
At the start: 4 copper layers, 75 x 44 mm, 34 parts, among them J1 USB-C 2.0, J2 microSD, J3 FPC 0.5mm 24p to SC3336, U1 Core1106 (RV1106G3), U2 USBLC6-2SC6

Commit message: Fix DRC errors; set via rules to JLC 4-layer limits
- Via rules: min diameter 0.45, min hole 0.2, min annular 0.075 mm
  (JLC's no-extra-cost tier). Clears 135 errors on the 0.45/0.25 GND
  stitching vias.
- Remove a stray no-net via off the board edge and a zero-length
  NPOR_RST track.
- Move TP2 0.4 mm right to clear the C8 courtyard.
- Fix starved thermals: GND tie tracks on C8.2 and U1.55, solid zone
  connection on R8.2.
- Refill zones.
- Includes in-progress schematic and board edits.

Co-Authored-By: Claude Opus 5.5 <noreply@anthropic.com>
Parts:
- moved C1 0.53 mm to (12.8, 29.1)
- moved F1 0.40 mm to (8.60, 29.5)
- moved TP2 0.40 mm to (55.4, 11.0)
Routing:
- net SD_D3: track 0.00 -> 18.0 mm
- net +5V: track 118.2 -> 107.9 mm, vias 10 -> 9
- net GND: track 67.8 -> 75.3 mm, vias 41 -> 85
- net USB_DM_CON: track 16.0 -> 12.5 mm
- net VBUS_DET: track 10.6 -> 13.7 mm
- net SD_D2: track 19.9 -> 17.3 mm
- net RECOV_HDR: track 77.1 -> 74.9 mm
- net SD_CMD: track 15.7 -> 13.8 mm
- net LED_A: track 5.52 -> 4.26 mm
- net SD_D1: track 15.9 -> 16.6 mm
- net LED_STAT: track 15.0 -> 14.3 mm
- added copper zone on In2.Cu, net +3V3
- added copper zone on In2.Cu, net +5V
- added copper zone on In2.Cu, net GND
- added copper zone on In2.Cu, net VBUS_IN
