File: hardware/LocalCam1.kicad_pcb (KiCad board)
At the start: 4 copper layers, 75 x 44 mm, 34 parts, among them J1 USB-C 2.0, J2 microSD, J3 FPC 0.5mm 24p to SC3336, U1 Core1106 (RV1106G3), U2 USBLC6-2SC6

Commit message: AAAAA it should cook a bit more now
Routing:
- net +5V: track 107.9 -> 120.8 mm
- net +1V8: track 69.9 -> 73.6 mm
- net SD_D2: track 17.3 -> 18.7 mm
- net GND: track 75.3 -> 73.9 mm, vias 85 -> 78
- net SD_CMD: track 13.8 -> 14.4 mm
Other:
- outline, holes or cut-outs redrawn

Commit message: fin
Routing:
- net +3V3: track 143.1 -> 145.0 mm
- net SD_D3: track 18.0 -> 18.9 mm
- net GND: vias 78 -> 85
