File: hardware/LocalCam1.kicad_sch (KiCad schematic)
At the start: 34 parts, among them J1 USB-C 2.0, J2 microSD (DM3AT), J3 FPC 0.5mm 24p to SC3336, U1 Core1106 (RV1106G3), U2 USBLC6-2SC6

Commit message: Fix DRC errors; set via rules to JLC 4-layer limits
- Via rules: min diameter 0.45, min hole 0.2, min annular 0.075 mm
  (JLC's no-extra-cost tier). Clears 135 errors on the 0.45/0.25 GND
  stitching vias.
- Remove a stray no-net via off the board edge and a zero-length
  NPOR_RST track.
- Move TP2 0.4 mm right to clear the C8 courtyard.
- Fix starved thermals: GND tie tracks on C8.2 and U1.55, solid zone
  connection on R8.2.
- Refill zones.
- Includes in-progress schematic and board edits.

Co-Authored-By: Claude Opus 5.5 <noreply@anthropic.com>
Parts:
- U1: value Core1106 (RV1106G3) -> ≈
Connections:
- net CC1: no longer names the net of J1.A5 (CC1), R1.1
- net CC2: no longer names the net of J1.B5 (CC2), R2.1
- net USB_DM_CON: no longer names the net of J1.A7 (D-), J1.B7 (D-), U2.1 (I/O1)
- net USB_DP_CON: no longer names the net of J1.A6 (D+), J1.B6 (D+), U2.3 (I/O2)
- net VBUS_IN: no longer names the net of F1.1, J1.A4 (VBUS), J1.A9 (VBUS), J1.B4 (VBUS), J1.B9 (VBUS)
Other:
- moved on the sheet: C3, C5, C6, D1, F1, R1, R2, R4, R9, U2
